Commit message: launch update

File: sid_ws/src/walle_description/urdf/walle.xacro (robot description, xacro)
@@ -92,5 +92,5 @@
   </collision>
 </link>
-<link name="lidar_1">
+<link name="laser_link">
   <inertial>
     <origin xyz="-7.153065918145268e-08 -1.1170202091591308e-07 0.009718373123905694" rpy="0 0 0"/>
@@ -112,5 +112,5 @@
   </collision>
 </link>
-<link name="imu_1">
+<link name="imu_link">
   <inertial>
     <origin xyz="-7.153065904527689e-08 1.3403373669393544e-07 -0.0024998122926913197" rpy="0 0 0"/>
@@ -136,5 +136,5 @@
   <parent link="base_link"/>
   <child link="left_wheel_1"/>
-  <axis xyz="-0.0 1.0 0.0"/>
+  <axis xyz="0.0 1.0 0.0"/>
 </joint>
 <joint name="right_wheel_joint" type="continuous">
@@ -142,5 +142,5 @@
   <parent link="base_link"/>
   <child link="right_wheel_1"/>
-  <axis xyz="0.0 -1.0 -0.0"/>
+  <axis xyz="0.0 1.0 0.0"/>
 </joint>
 <joint name="caster_wheel_joint" type="fixed">
@@ -152,10 +152,10 @@
   <origin xyz="0.001383 0.00039 0.12600" rpy="0 0 0"/>
   <parent link="base_link"/>
-  <child link="lidar_1"/>
+  <child link="laser_link"/>
 </joint>
 <joint name="imu_joint" type="fixed">
   <origin xyz="-0.021117 0.000222 0.0600" rpy="0 0 0"/>
   <parent link="base_link"/>
-  <child link="imu_1"/>
+  <child link="imu_link"/>
 </joint>
 </robot>

File: sid_ws/src/walle_description/urdf/walle_gazebo.xacro (robot description, xacro)
@@ -1,42 +1,36 @@
 <?xml version="1.0" ?>
-<robot name="walle" xmlns:xacro="http://www.ros.org/wiki/xacro" >
-<xacro:property name="body_color" value="Gazebo/Silver" />
-<gazebo reference="base_link">
-  <material>${body_color}</material>
-  <mu1>0.2</mu1>
-  <mu2>0.2</mu2>
-  <self_collide>true</self_collide>
-  <gravity>true</gravity>
-</gazebo>
-<gazebo reference="left_wheel_1">
-  <material>${body_color}</material>
-  <mu1>0.2</mu1>
-  <mu2>0.2</mu2>
-  <self_collide>true</self_collide>
-</gazebo>
-<gazebo reference="right_wheel_1">
-  <material>${body_color}</material>
-  <mu1>0.2</mu1>
-  <mu2>0.2</mu2>
-  <self_collide>true</self_collide>
-</gazebo>
-<gazebo reference="caster_wheel_1">
-  <material>${body_color}</material>
-  <mu1>0.2</mu1>
-  <mu2>0.2</mu2>
-  <self_collide>true</self_collide>
-</gazebo>
-<gazebo reference="lidar_1">
-  <material>${body_color}</material>
-  <mu1>0.2</mu1>
-  <mu2>0.2</mu2>
-  <self_collide>true</self_collide>
-</gazebo>
-<gazebo reference="imu_1">
-  <material>${body_color}</material>
-  <mu1>0.2</mu1>
-  <mu2>0.2</mu2>
-  <self_collide>true</self_collide>
-</gazebo>
+<robot name="walle" xmlns:xacro="http://www.ros.org/wiki/xacro">
+  <xacro:property name="body_color" value="Gazebo/silver" />
+  <xacro:property name="wheel_color" value="Gazebo/silver" />
+  <gazebo reference="left_wheel_1">
+    <material>${wheel_color}</material>
+    <mu1>1000000000000000.0</mu1>
+    <mu2>1000000000000000.0</mu2>
+    <kp>1000000000000.0</kp>
+    <kd>10.0</kd>
+    <minDepth>0.001</minDepth>
+    <maxVel>0.1</maxVel>
+    <fdir1>1 0 0</fdir1>
+  </gazebo>
+  <gazebo reference="right_wheel_1">
+    <material>${wheel_color}</material>
+    <mu1>1000000000000000.0</mu1>
+    <mu2>1000000000000000.0</mu2>
+    <kp>1000000000000.0</kp>
+    <kd>10.0</kd>
+    <minDepth>0.001</minDepth>
+    <maxVel>0.1</maxVel>
+    <fdir1>1 0 0</fdir1>
+  </gazebo>
+  <gazebo reference="caster_wheel_1">
+    <material>${body_color}</material>
+    <mu1>0.1</mu1>
+    <mu2>0.1</mu2>
+    <kp>1000000.0</kp>
+    <kd>100.0</kd>
+    <minDepth>0.001</minDepth>
+    <maxVel>0.1</maxVel>
+  </gazebo>
+<!-- ROS2 humble-->
   <gazebo>
     <xacro:if value="$(arg is_ignition)">
@@ -50,9 +44,10 @@
       </plugin>
     </xacro:if>
+<!-- ROS2 iron or above-->
     <xacro:unless value="$(arg is_ignition)">
       <plugin filename="gz_ros2_control-system" name="gz_ros2_control::GazeboSimROS2ControlPlugin">
         <parameters>$(find walle_controller)/config/walle_controllers.yaml</parameters>
       </plugin>
-       <plugin filename="gz-sim-imu-system" name="gz::sim::systems::Imu">
+      <plugin filename="gz-sim-imu-system" name="gz::sim::systems::Imu">
       </plugin>
       <plugin filename="gz-sim-sensors-system" name="gz::sim::systems::Sensors">
@@ -61,55 +56,56 @@
     </xacro:unless>
   </gazebo>
-  <gazebo reference="imu_1">
-   <sensor name="imu" type="imu">
-     <always_on>true</always_on>
-     <update_rate>100</update_rate>
-     <gz_frame_id>imu_1</gz_frame_id>
-     <topic>imu</topic>
-     <imu>
-      <angular_velocity>
-        <x>
-          <noise type="gaussian">
-            <mean>0.0</mean>
-            <stddev>2e-4</stddev>
-          </noise>
-        </x>
-        <y>
-          <noise type="gaussian">
-            <mean>0.0</mean>
-            <stddev>2e-4</stddev>
-          </noise>
-        </y>
-        <z>
-          <noise type="gaussian">
-            <mean>0.0</mean>
-            <stddev>2e-4</stddev>
-          </noise>
-        </z>
-      </angular_velocity>
-      <linear_acceleration>
-        <x>
-          <noise type="gaussian">
-            <mean>0.0</mean>
-            <stddev>1.7e-2</stddev>
-          </noise>
-        </x>
-        <y>
-          <noise type="gaussian">
-            <mean>0.0</mean>
-            <stddev>1.7e-2</stddev>
-          </noise>
-        </y>
-        <z>
-          <noise type="gaussian">
-            <mean>0.0</mean>
-            <stddev>1.7e-2</stddev>
-          </noise>
-        </z>
-      </linear_acceleration>
-    </imu>
-   </sensor>
+  <gazebo reference="imu_link">
+    <sensor name="imu" type="imu">
+      <always_on>true</always_on>
+      <update_rate>100</update_rate>
+      <gz_frame_id>imu_link</gz_frame_id>
+      <topic>imu</topic>
+      <imu>
+        <angular_velocity>
+          <x>
+            <noise type="gaussian">
+              <mean>0.0</mean>
+              <stddev>2e-4</stddev>
+            </noise>
+          </x>
+          <y>
+            <noise type="gaussian">
+              <mean>0.0</mean>
+              <stddev>2e-4</stddev>
+            </noise>
+          </y>
+          <z>
+            <noise type="gaussian">
+              <mean>0.0</mean>
+              <stddev>2e-4</stddev>
+            </noise>
+          </z>
+        </angular_velocity>
+        <linear_acceleration>
+          <x>
+            <noise type="gaussian">
+              <mean>0.0</mean>
+              <stddev>1.7e-2</stddev>
+            </noise>
+          </x>
+          <y>
+            <noise type="gaussian">
+              <mean>0.0</mean>
+              <stddev>1.7e-2</stddev>
+              </noise>
+          </y>
+          <z>
+            <noise type="gaussian">
+              <mean>0.0</mean>
+              <stddev>1.7e-2</stddev>
+              </noise>
+          </z>
+        </linear_acceleration>
+      </imu>
+    </sensor>
   </gazebo>
-  <gazebo reference="lidar_1">
+ <!-- 2D Laser Sensor -->
+  <gazebo reference="laser_link">
     <sensor name="lidar" type="gpu_lidar">
       <always_on>true</always_on>
@@ -117,5 +113,5 @@
       <topic>scan</topic>
       <update_rate>5</update_rate>
-      <gz_frame_id>lidar_1</gz_frame_id>
+      <gz_frame_id>laser_link</gz_frame_id>
       <lidar>
         <scan>
@@ -128,5 +124,5 @@
         </scan>
         <range>
-          <min>0.200000</min>
+          <min>0.20</min>
           <max>12.0</max>
           <resolution>0.02</resolution>
@@ -137,5 +133,5 @@
           <stddev>0.01</stddev>
         </noise>
-        </lidar>
+      </lidar>
     </sensor>
   </gazebo>

File: sid_ws/src/walle_description/urdf/walle_ros2_control.xacro (robot description, xacro)
@@ -2,22 +2,25 @@
 <robot name="walle" xmlns:xacro="http://www.ros.org/wiki/xacro" >
     <ros2_control name="RobotSystem" type="system">
+        <!-- ros2_control Gazebo -->
         <xacro:if value="$(arg is_sim)">
-          <xacro:if value="$(arg is_ignition)">
-            <hardware>
-                <plugin>ign_ros2_control/IgnitionSystem</plugin>
-            </hardware>
-          </xacro:if>
-           <xacro:unless value="$(arg is_ignition)">
-            <hardware>
-                <plugin>gz_ros2_control/GazeboSimSystem</plugin>
-            </hardware>
-           </xacro:unless>
+            <xacro:if value="$(arg is_ignition)">
+                <hardware>
+                    <plugin>ign_ros2_control/IgnitionSystem</plugin>
+                </hardware>
+            </xacro:if>
+            <xacro:unless value="$(arg is_ignition)">
+                <hardware>
+                    <plugin>gz_ros2_control/GazeboSimSystem</plugin>
+                </hardware>
+            </xacro:unless>
         </xacro:if>
+        <!-- ros2_control Real Robot -->
         <xacro:unless value="$(arg is_sim)">
             <hardware>
-                <plugin>walle_firmware/walleInterface</plugin>
+                <plugin>walle_firmware/WalleInterface</plugin>
                 <param name="port">/dev/ttyUSB0</param>
             </hardware>
         </xacro:unless>
+        <!-- ros2_control Common Interfaces -->
         <joint name="left_wheel_joint">
         <command_interface name="velocity">
